Commit message: Update sumo robot URDF with final sensor positions and components

File: urdf/sumo.urdf.xacro (robot description, xacro)
@@ -1,13 +1,26 @@
 <?xml version="1.0"?>
 <robot name="sumo_robot" xmlns:xacro="http://www.ros.org/wiki/xacro">
+    <material name="grey">
+        <color rgba="0.6 0.6 0.6 1.0"/>
+    </material>
+    <material name="black">
+        <color rgba="0.1 0.1 0.1 1.0"/>
+    </material>
+    <link name="base_link"/>
+    <joint name="base_joint" type="fixed">
+        <parent link="base_link"/>
+        <child link="body"/>
+        <origin xyz="0 0 0" rpy="1.5708 0 0"/>
+    </joint>
     <link name="body">
         <visual>
             <geometry>
-               <mesh filename="package://sumo_description/meshes/STLs/body.STL" scale="0.001 0.001 0.001"/>
-            </geometry>
-        </visual>
-        <collision>
-            <geometry>
-                <mesh filename="package://sumo_description/meshes/STLs/body.STL" scale="0.001 0.001 0.001"/>
+             <mesh filename="package://sumo_description/meshes/STLs/bodyhhh.STL" scale="1 1 1"/>
+            </geometry>
+            <material name="grey"/>
+        </visual>
+        <collision>
+            <geometry>
+                <mesh filename="package://sumo_description/meshes/STLs/bodyhhh.STL" scale="1 1 1"/>
             </geometry>
         </collision>
@@ -18,21 +31,40 @@
       </inertial>
     </link>
+    <link name="cutting_wheel_connector">
+        <visual>
+            <origin xyz="0 0 -0.02" rpy="0 0 0"/>
+            <geometry>
+                <cylinder radius="0.015" length="0.04"/>
+            </geometry>
+            <material name="black"/>
+        </visual>
+        <inertial>
+            <mass value="0.001"/>
+            <inertia ixx="0.000001" ixy="0.0" ixz="0.0" iyy="0.000001" iyz="0.0" izz="0.000001"/>
+        </inertial>
+    </link>
+    <joint name="cutting_wheel_connector_joint" type="fixed">
+        <parent link="body"/>
+        <child link="cutting_wheel_connector"/>
+        <origin xyz="0.003 0.08986 0.09845" rpy="-1.0472 0 0"/>
+    </joint>
     <link name="cutting_wheel">
         <visual>
-            <origin xyz="-0.014 -0.124 -0.073" rpy="0 0 0"/>
-            <geometry>
-               <mesh filename="package://sumo_description/meshes/STLs/cutting_wheel_final.STL" scale="0.001 0.001 0.001"/>
-            </geometry>
-        </visual>
-        <collision>
-            <origin xyz="-0.014 -0.124 -0.073" rpy="0 0 0"/>
-            <geometry>
-                <cylinder radius="0.106" length="0.01"/>
-            </geometry>
-        </collision>
-        <inertial>
-            <origin xyz="0.01938 0.10888 0.08419" rpy="0 0 0"/>
+            <origin xyz="0 0 0" rpy="0 0 0"/>
+            <geometry>
+            <mesh filename="package://sumo_description/meshes/STLs/Cutting_wheelfffhh.STL" scale="1 1 1"/>
+            </geometry>
+            <material name="black"/>
+        </visual>
+        <collision>
+            <origin xyz="0 0 0" rpy="0 0 0"/>
+            <geometry>
+                <cylinder radius="0.135" length="0.004"/>
+            </geometry>
+        </collision>
+        <inertial>
+            <origin xyz="0 0 0.00294" rpy="0 0 0"/>
             <mass value="0.17182"/>
-            <inertia ixx="0.000470" ixy="0.0" ixz="0.0" iyy="0.000821" iyz="-0.000202" izz="0.000587"/>
+            <inertia ixx="0.000474" ixy="0.0" ixz="0.0" iyy="0.000474" iyz="0.0" izz="0.000947"/>
         </inertial>
     </link>
@@ -40,7 +72,155 @@
         <parent link="body"/>
         <child link="cutting_wheel"/>
-        <origin xyz="0.003 0.08986 0.09845" rpy="0 0.52359 0"/>
+        <origin xyz="0.003 0.08986 0.09845" rpy="-1.0472 0 0"/>
         <axis xyz="0 0 1"/>
         <limit effort="500.0" velocity="20.0"/>
     </joint>
+    <link name="right_wheel">
+        <visual>
+            <origin xyz="0 0 0" rpy="0 0 0"/>
+            <geometry>
+                <mesh filename="package://sumo_description/meshes/STLs/Wheelh.STL" scale="1 1 1"/>
+            </geometry>
+            <material name="black"/>
+        </visual>
+        <collision>
+            <origin xyz="0 0 0" rpy="0 1.5708 0"/>
+            <geometry>
+                <cylinder radius="0.0425" length="0.038"/>
+            </geometry>
+        </collision>
+        <inertial>
+            <origin xyz="0 0 0" rpy="0 0 0"/>
+            <mass value="0.10621"/>
+            <inertia ixx="0.000108" ixy="0.0" ixz="0.0" iyy="0.000061" iyz="0.0" izz="0.000061"/>
+        </inertial>
+    </link>
+    <joint name="right_wheel_joint" type="continuous">
+        <parent link="body"/>
+        <child link="right_wheel"/>
+        <origin xyz="0.104029 0.031999 -0.063999" rpy="0 0 0"/>
+        <axis xyz="1 0 0"/>
+        <limit effort="500.0" velocity="20.0"/>
+    </joint>
+    <link name="left_wheel">
+        <visual>
+            <origin xyz="0 0 0" rpy="0 0 0"/>
+            <geometry>
+                <mesh filename="package://sumo_description/meshes/STLs/Wheelh.STL" scale="1 1 1"/>
+            </geometry>
+            <material name="black"/>
+        </visual>
+        <collision>
+            <origin xyz="0 0 0" rpy="0 1.5708 0"/>
+            <geometry>
+                <cylinder radius="0.0425" length="0.038"/>
+            </geometry>
+        </collision>
+        <inertial>
+            <origin xyz="0 0 0" rpy="0 0 0"/>
+            <mass value="0.10621"/>
+            <inertia ixx="0.000108" ixy="0.0" ixz="0.0" iyy="0.000061" iyz="0.0" izz="0.000061"/>
+        </inertial>
+    </link>
+    <joint name="left_wheel_joint" type="continuous">
+        <parent link="body"/>
+        <child link="left_wheel"/>
+        <origin xyz="-0.104029 0.031999 -0.063999" rpy="0 0 0"/>
+        <axis xyz="1 0 0"/>
+        <limit effort="500.0" velocity="20.0"/>
+    </joint>
+    <link name="camera_link">
+        <visual>
+            <origin xyz="0 0 0" rpy="0 0 0"/>
+            <geometry>
+                <mesh filename="package://sumo_description/meshes/STLs/WebCamhh.STL" scale="1 1 1"/>
+            </geometry>
+            <material name="black"/>
+        </visual>
+        <collision>
+            <origin xyz="0 0 0" rpy="0 0 0"/>
+            <geometry>
+                <box size="0.077 0.023 0.029"/>
+            </geometry>
+        </collision>
+    </link>
+    <joint name="camera_joint" type="fixed">
+        <parent link="body"/>
+        <child link="camera_link"/>
+        <origin xyz="0.000210 0.170350 -0.169" rpy="5.6416 0 0"/>
+    </joint>
+    <link name="lidar_link">
+        <visual>
+            <origin xyz="0 0 0" rpy="0 0 0"/>
+            <geometry>
+                <box size="0.03 0.03 0.03"/>
+            </geometry>
+            <material name="black"/>
+        </visual>
+        <collision>
+            <origin xyz="0 0 0" rpy="0 0 0"/>
+            <geometry>
+                <box size="0.01 0.01 0.01"/>
+            </geometry>
+        </collision>
+        <inertial>
+            <mass value="0.05"/>
+            <inertia ixx="0.00001" ixy="0.0" ixz="0.0" iyy="0.00001" iyz="0.0" izz="0.00001"/>
+        </inertial>
+    </link>
+      <joint name="lidar_joint" type="fixed">
+        <parent link="body"/>
+        <child link="lidar_link"/>
+        <origin xyz="0.000210 0.20 -0.174" rpy="0 0 0"/>
+      </joint>
+    <link name="caster_link">
+        <visual>
+            <origin xyz="0 0 0" rpy="0 0 0"/>
+            <geometry>
+                <box size="0.02 0.02 0.02"/>
+            </geometry>
+            <material name="black"/>
+        </visual>
+        <collision>
+            <origin xyz="0 0 0" rpy="0 0 0"/>
+            <geometry>
+                <box size="0.02 0.02 0.02"/>
+            </geometry>
+        </collision>
+        <inertial>
+            <mass value="0.05"/>
+            <inertia ixx="0.00001" ixy="0.0" ixz="0.0" iyy="0.00001" iyz="0.0" izz="0.00001"/>
+        </inertial>
+    </link>
+    <joint name="caster_joint" type="fixed">
+        <parent link="body"/>
+        <child link="caster_link"/>
+        <origin xyz="0 0 0.08" rpy="0 0 0"/>
+    </joint>
+    <gazebo reference="caster_link">
+        <mu1 value="0.0"/>
+        <mu2 value="0.0"/>
+        <material>Gazebo/Black</material>
+    </gazebo>
+    <link name="imu_link">
+    </link>
+    <joint name="imu_joint" type="fixed">
+        <parent link="body"/>
+        <child link="imu_link"/>
+        <origin xyz="0 0 0" rpy="0 0 0"/>
+    </joint>
+    <gazebo reference="right_wheel">
+        <mu1 value="200.0"/>
+        <mu2 value="100.0"/>
+        <kp value="10000000.0"/>
+        <kd value="1.0"/>
+        <material>Gazebo/Black</material>
+    </gazebo>
+    <gazebo reference="left_wheel">
+        <mu1 value="200.0"/>
+        <mu2 value="100.0"/>
+        <kp value="10000000.0"/>
+        <kd value="1.0"/>
+        <material>Gazebo/Black</material>
+    </gazebo>
 </robot>
